File: Hardware/VoltageRegulator/VoltageRegulator.kicad_pcb (KiCad board)
At the start: 2 copper layers, 22.1 x 14.2 mm, 10 parts, among them J1 Conn_01x04, U1 TPS7A2501DRVR

Commit message: Neaten up schematic, add precision designators for resistors
Parts:
- R1: value 360K -> 360K 1%
- R2: value 3M -> 3M 1%
- R3: value 1M -> 1M 1%
Changed lines of the file:
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@@
         (effects (font (size 1 1) (thickness 0.15)))
     )
-    (fp_text value "3M" (at -4.762 0) (layer "F.Fab")
+    (fp_text value "3M 1%" (at -4.762 0) (layer "F.Fab")
         (effects (font (size 1 1) (thickness 0.15)))
     )
@@
         (effects (font (size 1 1) (thickness 0.15)))
     )
-    (fp_text value "1M" (at 4.763 0) (layer "F.Fab")
+    (fp_text value "1M 1%" (at 4.763 0) (layer "F.Fab")
         (effects (font (size 1 1) (thickness 0.15)))
     )
@@
         (effects (font (size 1 1) (thickness 0.15)))
     )
-    (fp_text value "360K" (at 5.905 0) (layer "F.Fab")
-        (effects (font (size 1 1) (thickness 0.15)))
-    )
+    (fp_text value "360K 1%" (at 5.905 0) (layer "F.Fab")
+        (effects (font (size 1 1) (thickness 0.15)))
+    )
